File: HW/ClockOmat.kicad_pcb (KiCad board)
At the start: 2 copper layers, 30.5 x 114.3 mm, 90 parts, among them J1 EurorackPower, Q1 BC817, Q10 BC807, Q11 BC817, Q12 BC817, Q2 BC817, Q3 BC817, Q4 BC817, Q5 BC817, Q6 BC817, Q7 BC817, Q8 BC807, Q9 BC807, SW1 Rotary_Encoder_Switch, SW2 SW_Push, SW3 SW_Push, U1 ATmega328P-AU, U2 MCP23S08-SSOP, U3 CA56-12EWA, U5 L7805, Y1 Crystal

Commit message: some error corrections
Parts:
- added C9: 100nF, Capacitor_SMD:C_0805_2012Metric_Pad1.18x1.45mm_HandSolder, F.Cu at (168.8, 65.0)
- added R43: 47K, Resistor_SMD:R_0805_2012Metric_Pad1.20x1.40mm_HandSolder, F.Cu at (166.5, 80.0)
- U2: value MCP23S08-SSOP -> MCP23S08-xSS-20; footprint Package_SO:SSOP-18_4.4x6.5mm_P0.65mm -> Package_SO:SSOP-20_5.3x7.2mm_P0.65mm
- moved R33 2.44 mm to (173.2, 36.3), turned to 0 degrees
- moved R29 1.50 mm to (172.2, 34.4)
- moved R26 0.51 mm to (173.2, 41.4)
- moved U2 0.48 mm to (179.0, 38.7)
- moved C6 0.44 mm to (169.1, 68.0)
- moved Q10 0.16 mm to (169.6, 41.5)
Connections:
- R40 pad 1: +5V -> Net-(R40-Pad1)
- SW2 pad 1: +5V -> Net-(R40-Pad1)
- U2 pad 10: c -> (no net)
- U2 pad 11: g -> (no net)
- U2 pad 12: p -> c
- U2 pad 13: d -> g
- U2 pad 14: e -> p
- U2 pad 15: a -> d
- U2 pad 16: f -> e
- U2 pad 17: b -> a
- U2 pad 18: +5V -> f
Routing:
- net Net-(R40-Pad1): track 0.00 -> 24.1 mm
- net +5V: track 136.4 -> 146.7 mm, vias 7 -> 8
- net c: track 2.69 -> 4.86 mm
- net GNDD: track 337.8 -> 339.6 mm
- net Net-(R32-Pad1): track 10.2 -> 11.5 mm
- net Net-(R28-Pad1): track 2.57 -> 3.84 mm
- net Net-(R27-Pad1): track 4.48 -> 5.75 mm
- net D1: track 5.16 -> 3.89 mm
- net f: track 7.61 -> 6.42 mm
- net b: track 9.07 -> 7.88 mm
- net g: track 3.32 -> 4.35 mm
- net Net-(R29-Pad1): track 3.75 -> 4.67 mm
- net Net-(Q10-Pad1): track 2.44 -> 1.80 mm
- net Net-(R34-Pad1): track 2.19 -> 2.72 mm
- net Net-(R30-Pad1): track 2.19 -> 2.72 mm
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Other:
- rule trace_min: 0.2 -> 0.15
